File: NumPad.sch (KiCad schematic (older format))
At the start: 112 parts, among them J1 Micro_SD_Card_Det, J2 OLED1, J3 OLED2, J4 Conn_01x05_Female, SW1 SW_SPST, SW10 SW_SPST, SW11 SW_SPST, SW12 SW_SPST, SW13 SW_SPST, SW14 SW_SPST, SW15 SW_SPST, SW16 SW_SPST, SW17 SW_SPST, SW18 SW_SPST, SW19 SW_SPST, SW2 SW_SPST, SW20 SW_SPST, SW21 SW_SPST, SW22 SW_SPST, SW23 SW_SPST, SW24 SW_SPST, SW25 SW_BUTTONRESET, SW26 SW_BUTTON2, SW27 SW_BUTTON1, SW28 SW_BOOT0, SW29 Rotary_Encoder_Switch, SW3 SW_SPST, SW4 SW_SPST, SW5 SW_SPST, SW6 SW_SPST, SW7 SW_SPST, SW8 SW_SPST, SW9 SW_SPST, U1 LM117_TO3, U2 STM32F072C8Tx, U3 74AHCT1G08

Commit message: update
Parts:
- SW1, SW10, SW11, SW12, SW13, SW14, SW15, SW16, SW17, SW18, SW19, SW2, SW20, SW21, SW22, SW23, SW24, SW3, SW4, SW5, SW6, SW7, SW8, SW9: footprint MX_Only:MXOnly-1U -> MX_Only:MXOnly-1U-NoLED
- U1: footprint Package_TO_SOT_THT:TO-3 -> Package_TO_SOT_SMD:SOT-23-5_HandSoldering
Changed lines of the file:
@@
 F 0 "U1" H 1275 3042 50  0000 C CNN
 F 1 "LM117_TO3" H 1275 2951 50  0000 C CNN
-F 2 "Package_TO_SOT_THT:TO-3" H 1275 3000 50  0001 C CIN
+F 2 "Package_TO_SOT_SMD:SOT-23-5_HandSoldering" H 1275 3000 50  0001 C CIN
 F 3 "http://www.ti.com/lit/ds/symlink/lm317.pdf" H 1275 2800 50  0001 C CNN
 	1    1275 2800
@@
 F 0 "SW1" H 8725 1334 50  0000 C CNN
 F 1 "SW_SPST" H 8725 1243 50  0000 C CNN
-F 2 "MX_Only:MXOnly-1U" H 8725 1100 50  0001 C CNN
+F 2 "MX_Only:MXOnly-1U-NoLED" H 8725 1100 50  0001 C CNN
 F 3 "~" H 8725 1100 50  0001 C CNN
 	1    8725 1100
@@
 F 0 "SW2" H 8725 1959 50  0000 C CNN
 F 1 "SW_SPST" H 8725 1868 50  0000 C CNN
-F 2 "MX_Only:MXOnly-1U" H 8725 1725 50  0001 C CNN
+F 2 "MX_Only:MXOnly-1U-NoLED" H 8725 1725 50  0001 C CNN
 F 3 "~" H 8725 1725 50  0001 C CNN
 	1    8725 1725
@@
 F 0 "SW3" H 8725 2584 50  0000 C CNN
 F 1 "SW_SPST" H 8725 2493 50  0000 C CNN
-F 2 "MX_Only:MXOnly-1U" H 8725 2350 50  0001 C CNN
+F 2 "MX_Only:MXOnly-1U-NoLED" H 8725 2350 50  0001 C CNN
 F 3 "~" H 8725 2350 50  0001 C CNN
 	1    8725 2350
@@
 F 0 "SW4" H 8725 3209 50  0000 C CNN
 F 1 "SW_SPST" H 8725 3118 50  0000 C CNN
-F 2 "MX_Only:MXOnly-1U" H 8725 2975 50  0001 C CNN
+F 2 "MX_Only:MXOnly-1U-NoLED" H 8725 2975 50  0001 C CNN
 F 3 "~" H 8725 2975 50  0001 C CNN
 	1    8725 2975
@@
 F 0 "SW5" H 8725 3809 50  0000 C CNN
 F 1 "SW_SPST" H 8725 3718 50  0000 C CNN
-F 2 "MX_Only:MXOnly-1U" H 8725 3575 50  0001 C CNN
+F 2 "MX_Only:MXOnly-1U-NoLED" H 8725 3575 50  0001 C CNN
 F 3 "~" H 8725 3575 50  0001 C CNN
 	1    8725 3575
@@
 F 0 "SW6" H 8725 4434 50  0000 C CNN
 F 1 "SW_SPST" H 8725 4343 50  0000 C CNN
-F 2 "MX_Only:MXOnly-1U" H 8725 4200 50  0001 C CNN
+F 2 "MX_Only:MXOnly-1U-NoLED" H 8725 4200 50  0001 C CNN
 F 3 "~" H 8725 4200 50  0001 C CNN
 	1    8725 4200
@@
 F 0 "SW7" H 9375 1334 50  0000 C CNN
 F 1 "SW_SPST" H 9375 1243 50  0000 C CNN
-F 2 "MX_Only:MXOnly-1U" H 9375 1100 50  0001 C CNN
+F 2 "MX_Only:MXOnly-1U-NoLED" H 9375 1100 50  0001 C CNN
 F 3 "~" H 9375 1100 50  0001 C CNN
 	1    9375 1100
@@
 F 0 "SW8" H 9375 1959 50  0000 C CNN
 F 1 "SW_SPST" H 9375 1868 50  0000 C CNN
-F 2 "MX_Only:MXOnly-1U" H 9375 1725 50  0001 C CNN
+F 2 "MX_Only:MXOnly-1U-NoLED" H 9375 1725 50  0001 C CNN
 F 3 "~" H 9375 1725 50  0001 C CNN
 	1    9375 1725
@@
 F 0 "SW9" H 9375 2584 50  0000 C CNN
 F 1 "SW_SPST" H 9375 2493 50  0000 C CNN
-F 2 "MX_Only:MXOnly-1U" H 9375 2350 50  0001 C CNN
+F 2 "MX_Only:MXOnly-1U-NoLED" H 9375 2350 50  0001 C CNN
 F 3 "~" H 9375 2350 50  0001 C CNN
 	1    9375 2350
@@
 F 0 "SW10" H 9375 3209 50  0000 C CNN
 F 1 "SW_SPST" H 9375 3118 50  0000 C CNN
-F 2 "MX_Only:MXOnly-1U" H 9375 2975 50  0001 C CNN
+F 2 "MX_Only:MXOnly-1U-NoLED" H 9375 2975 50  0001 C CNN
 F 3 "~" H 9375 2975 50  0001 C CNN
 	1    9375 2975
@@
 F 0 "SW11" H 9375 3809 50  0000 C CNN
 F 1 "SW_SPST" H 9375 3718 50  0000 C CNN
-F 2 "MX_Only:MXOnly-1U" H 9375 3575 50  0001 C CNN
+F 2 "MX_Only:MXOnly-1U-NoLED" H 9375 3575 50  0001 C CNN
 F 3 "~" H 9375 3575 50  0001 C CNN
 	1    9375 3575
@@
 F 0 "SW12" H 9375 4434 50  0000 C CNN
 F 1 "SW_SPST" H 9375 4343 50  0000 C CNN
-F 2 "MX_Only:MXOnly-1U" H 9375 4200 50  0001 C CNN
+F 2 "MX_Only:MXOnly-1U-NoLED" H 9375 4200 50  0001 C CNN
 F 3 "~" H 9375 4200 50  0001 C CNN
 	1    9375 4200
@@
 F 0 "SW13" H 10025 1334 50  0000 C CNN
 F 1 "SW_SPST" H 10025 1243 50  0000 C CNN
-F 2 "MX_Only:MXOnly-1U" H 10025 1100 50  0001 C CNN
+F 2 "MX_Only:MXOnly-1U-NoLED" H 10025 1100 50  0001 C CNN
 F 3 "~" H 10025 1100 50  0001 C CNN
 	1    10025 1100
@@
 F 0 "SW14" H 10025 1959 50  0000 C CNN
 F 1 "SW_SPST" H 10025 1868 50  0000 C CNN
-F 2 "MX_Only:MXOnly-1U" H 10025 1725 50  0001 C CNN
+F 2 "MX_Only:MXOnly-1U-NoLED" H 10025 1725 50  0001 C CNN
 F 3 "~" H 10025 1725 50  0001 C CNN
 	1    10025 1725
@@
 F 0 "SW15" H 10025 2584 50  0000 C CNN
 F 1 "SW_SPST" H 10025 2493 50  0000 C CNN
-F 2 "MX_Only:MXOnly-1U" H 10025 2350 50  0001 C CNN
+F 2 "MX_Only:MXOnly-1U-NoLED" H 10025 2350 50  0001 C CNN
 F 3 "~" H 10025 2350 50  0001 C CNN
 	1    10025 2350
@@
 F 0 "SW16" H 10025 3209 50  0000 C CNN
 F 1 "SW_SPST" H 10025 3118 50  0000 C CNN
-F 2 "MX_Only:MXOnly-1U" H 10025 2975 50  0001 C CNN
+F 2 "MX_Only:MXOnly-1U-NoLED" H 10025 2975 50  0001 C CNN
 F 3 "~" H 10025 2975 50  0001 C CNN
 	1    10025 2975
@@
 F 0 "SW17" H 10025 3809 50  0000 C CNN
 F 1 "SW_SPST" H 10025 3718 50  0000 C CNN
-F 2 "MX_Only:MXOnly-1U" H 10025 3575 50  0001 C CNN
+F 2 "MX_Only:MXOnly-1U-NoLED" H 10025 3575 50  0001 C CNN
 F 3 "~" H 10025 3575 50  0001 C CNN
 	1    10025 3575
@@
 F 0 "SW18" H 10025 4434 50  0000 C CNN
 F 1 "SW_SPST" H 10025 4343 50  0000 C CNN
-F 2 "MX_Only:MXOnly-1U" H 10025 4200 50  0001 C CNN
+F 2 "MX_Only:MXOnly-1U-NoLED" H 10025 4200 50  0001 C CNN
 F 3 "~" H 10025 4200 50  0001 C CNN
 	1    10025 4200
@@
 F 0 "SW19" H 10675 1334 50  0000 C CNN
 F 1 "SW_SPST" H 10675 1243 50  0000 C CNN
-F 2 "MX_Only:MXOnly-1U" H 10675 1100 50  0001 C CNN
+F 2 "MX_Only:MXOnly-1U-NoLED" H 10675 1100 50  0001 C CNN
 F 3 "~" H 10675 1100 50  0001 C CNN
 	1    10675 1100
@@
 F 0 "SW20" H 10675 1959 50  0000 C CNN
 F 1 "SW_SPST" H 10675 1868 50  0000 C CNN
-F 2 "MX_Only:MXOnly-1U" H 10675 1725 50  0001 C CNN
+F 2 "MX_Only:MXOnly-1U-NoLED" H 10675 1725 50  0001 C CNN
 F 3 "~" H 10675 1725 50  0001 C CNN
 	1    10675 1725
@@
 F 0 "SW21" H 10675 2584 50  0000 C CNN
 F 1 "SW_SPST" H 10675 2493 50  0000 C CNN
-F 2 "MX_Only:MXOnly-1U" H 10675 2350 50  0001 C CNN
+F 2 "MX_Only:MXOnly-1U-NoLED" H 10675 2350 50  0001 C CNN
 F 3 "~" H 10675 2350 50  0001 C CNN
 	1    10675 2350
@@
 F 0 "SW22" H 10675 3209 50  0000 C CNN
 F 1 "SW_SPST" H 10675 3118 50  0000 C CNN
-F 2 "MX_Only:MXOnly-1U" H 10675 2975 50  0001 C CNN
+F 2 "MX_Only:MXOnly-1U-NoLED" H 10675 2975 50  0001 C CNN
 F 3 "~" H 10675 2975 50  0001 C CNN
 	1    10675 2975
@@
 F 0 "SW23" H 10675 3809 50  0000 C CNN
 F 1 "SW_SPST" H 10675 3718 50  0000 C CNN
-F 2 "MX_Only:MXOnly-1U" H 10675 3575 50  0001 C CNN
+F 2 "MX_Only:MXOnly-1U-NoLED" H 10675 3575 50  0001 C CNN
 F 3 "~" H 10675 3575 50  0001 C CNN
 	1    10675 3575
@@
 F 0 "SW24" H 10675 4434 50  0000 C CNN
 F 1 "SW_SPST" H 10675 4343 50  0000 C CNN
-F 2 "MX_Only:MXOnly-1U" H 10675 4200 50  0001 C CNN
+F 2 "MX_Only:MXOnly-1U-NoLED" H 10675 4200 50  0001 C CNN
 F 3 "~" H 10675 4200 50  0001 C CNN
 	1    10675 4200
