File: _autosave-NumPad.sch (KiCad schematic (older format))
At the start: 112 parts, among them J1 Micro_SD_Card_Det, J2 OLED1, J3 OLED2, J4 Conn_01x05_Female, SW1 SW_SPST, SW10 SW_SPST, SW11 SW_SPST, SW12 SW_SPST, SW13 SW_SPST, SW14 SW_SPST, SW15 SW_SPST, SW16 SW_SPST, SW17 SW_SPST, SW18 SW_SPST, SW19 SW_SPST, SW2 SW_SPST, SW20 SW_SPST, SW21 SW_SPST, SW22 SW_SPST, SW23 SW_SPST, SW24 SW_SPST, SW25 SW_BUTTONRESET, SW26 SW_BUTTON2, SW27 SW_BUTTON1, SW28 SW_BOOT0, SW29 Rotary_Encoder_Switch, SW3 SW_SPST, SW4 SW_SPST, SW5 SW_SPST, SW6 SW_SPST, SW7 SW_SPST, SW8 SW_SPST, SW9 SW_SPST, U1 LM117_TO3, U2 STM32F072C8Tx, U3 74AHCT1G08

Commit message: update PCB
Parts:
- D1: footprint Package_TO_SOT_SMD:SOT-143 -> random-keyboard-parts:SOT143B
Connections:
- net BUT1: now also U2.25 (PB12); no longer U2.38 (PA15)
- net ENC_SWITCH: now also U2.28 (PB15); no longer U2.39 (PB3)
- net POT_SLIDER: now also U2.27 (PB14); no longer U2.25 (PB12)
- net col3: now also U2.12 (PA2); no longer U2.3 (PC14)
- net row0: now also U2.13 (PA3); no longer U2.4 (PC15)
- net row1: now also U2.6 (PF1); no longer U2.5 (PF0)
- net row2: now also U2.5 (PF0); no longer U2.6 (PF1)
- net row3: now also U2.4 (PC15); no longer U2.45 (PB8)
- net row4: now also U2.3 (PC14); no longer U2.12 (PA2)
- net BUT2: now reaches R5.2, SW26.1
- net BUT2: now also U2.26 (PB13); no longer U2.13 (PA3)
Other:
- moved on the sheet: R5, SW26
Changed lines of the file:
@@
 F 0 "D1" V 3500 1750 50  0000 L CNN
 F 1 "PRTR5V0U2X" V 3400 1650 50  0000 L CNN
-F 2 "Package_TO_SOT_SMD:SOT-143" H 3285 1350 50  0001 C CNN
+F 2 "random-keyboard-parts:SOT143B" H 3285 1350 50  0001 C CNN
 F 3 "https://assets.nexperia.com/documents/data-sheet/PRTR5V0U2X.pdf" H 3285 1350 50  0001 C CNN
 	1    3225 1350
@@
 Wire Wire Line
 	3525 3700 2900 3700
+Text GLabel 2475 5800 2    60   Input ~ 0
+row0
+Text GLabel 1175 4900 0    60   Input ~ 0
+row1
+Text GLabel 1175 4800 0    60   Input ~ 0
+row2
 Text GLabel 1175 5300 0    60   Input ~ 0
-row0
-Text GLabel 1175 4800 0    60   Input ~ 0
-row1
-Text GLabel 1175 4900 0    60   Input ~ 0
-row2
-Text GLabel 1175 6300 0    60   Input ~ 0
 row3
 Text GLabel 2475 5500 2    60   Input ~ 0
@@
 L Switch:SW_Push SW26
 U 1 1 5E9524FE
-P 3550 6125
-F 0 "SW26" H 3550 6410 50  0000 C CNN
-F 1 "SW_BUTTON2" H 3550 6319 50  0000 C CNN
-F 2 "keyboard_parts:TactSwitch" H 3550 6325 50  0001 C CNN
-F 3 "~" H 3550 6325 50  0001 C CNN
-	1    3550 6125
+P 3850 6275
+F 0 "SW26" H 3850 6560 50  0000 C CNN
+F 1 "SW_BUTTON2" H 3850 6469 50  0000 C CNN
+F 2 "keyboard_parts:TactSwitch" H 3850 6475 50  0001 C CNN
+F 3 "~" H 3850 6475 50  0001 C CNN
+	1    3850 6275
 	1    0    0    -1
 $EndComp
@@
 L power:GND #PWR032
 U 1 1 5E953574
-P 3850 6125
-F 0 "#PWR032" H 3850 5875 50  0001 C CNN
-F 1 "GND" H 3855 5952 50  0000 C CNN
-F 2 "" H 3850 6125 50  0001 C CNN
-F 3 "" H 3850 6125 50  0001 C CNN
-	1    3850 6125
-	1    0    0    -1
-$EndComp
-Wire Wire Line
-	3850 6125 3750 6125
+P 4150 6275
+F 0 "#PWR032" H 4150 6025 50  0001 C CNN
+F 1 "GND" H 4155 6102 50  0000 C CNN
+F 2 "" H 4150 6275 50  0001 C CNN
+F 3 "" H 4150 6275 50  0001 C CNN
+	1    4150 6275
+	1    0    0    -1
+$EndComp
+Wire Wire Line
+	4150 6275 4050 6275
 $Comp
 L power:+3.3V #PWR027
 U 1 1 5E95E2CA
-P 3250 5825
-F 0 "#PWR027" H 3250 5675 50  0001 C CNN
-F 1 "+3.3V" H 3265 5998 50  0000 C CNN
-F 2 "" H 3250 5825 50  0001 C CNN
-F 3 "" H 3250 5825 50  0001 C CNN
-	1    3250 5825
+P 3550 5975
+F 0 "#PWR027" H 3550 5825 50  0001 C CNN
+F 1 "+3.3V" H 3565 6148 50  0000 C CNN
+F 2 "" H 3550 5975 50  0001 C CNN
+F 3 "" H 3550 5975 50  0001 C CNN
+	1    3550 5975
 	1    0    0    -1
 $EndComp
@@
 L Device:R_Small R5
 U 1 1 5E95E6BD
-P 3250 5925
-F 0 "R5" H 3100 6025 50  0000 L CNN
-F 1 "10K" H 3050 5925 50  0000 L CNN
-F 2 "Resistor_SMD:R_0603_1608Metric" H 3250 5925 50  0001 C CNN
-F 3 "~" H 3250 5925 50  0001 C CNN
-	1    3250 5925
-	1    0    0    -1
-$EndComp
-Wire Wire Line
-	2475 5800 2975 5800
+P 3550 6075
+F 0 "R5" H 3400 6175 50  0000 L CNN
+F 1 "10K" H 3350 6075 50  0000 L CNN
+F 2 "Resistor_SMD:R_0603_1608Metric" H 3550 6075 50  0001 C CNN
+F 3 "~" H 3550 6075 50  0001 C CNN
+	1    3550 6075
+	1    0    0    -1
+$EndComp
 $Comp
 L power:GND #PWR024
@@
 Wire Wire Line
 	10025 6175 10025 6375
-Text GLabel 1175 6700 0    60   Input ~ 0
+Text GLabel 1175 6900 0    60   Input ~ 0
 POT_SLIDER
 $Comp
@@
 Wire Wire Line
 	10525 6025 10175 6025
-Text GLabel 2475 5700 2    60   Input ~ 0
+Text GLabel 1175 5200 0    60   Input ~ 0
 row4
 Text GLabel 1175 5100 0    60   Input ~ 0
 row5
-Text GLabel 1175 5200 0    60   Input ~ 0
+Text GLabel 2475 5700 2    60   Input ~ 0
 col3
 Text GLabel 1175 6100 0    50   Input ~ 0
@@
 NoConn ~ 12950 150
 Wire Wire Line
-	2975 6125 3250 6125
-Wire Wire Line
-	2975 5800 2975 6125
-Wire Wire Line
-	3250 6125 3250 6025
-Connection ~ 3250 6125
-Wire Wire Line
-	3250 6125 3350 6125
+	3275 6275 3550 6275
+Wire Wire Line
+	3550 6275 3550 6175
+Connection ~ 3550 6275
+Wire Wire Line
+	3550 6275 3650 6275
 Wire Wire Line
 	3250 5325 3250 5075
@@
 	3250 5325 2950 5325
 Connection ~ 3250 5325
-Text GLabel 2475 7000 2    60   Input ~ 0
-BUT1
 $Comp
 L Device:Rotary_Encoder_Switch SW29
@@
 Wire Wire Line
 	9650 4650 9925 4650
-Text GLabel 1175 5800 0    50   Input ~ 0
+Text GLabel 1175 7000 0    50   Input ~ 0
 ENC_SWITCH
 Text GLabel 9650 4925 0    50   Input ~ 0
@@
 	1    0    0    -1
 $EndComp
-NoConn ~ 1175 6800
-NoConn ~ 1175 6900
-NoConn ~ 1175 7000
 NoConn ~ 2475 6300
 NoConn ~ 1175 5900
+Text GLabel 3275 6275 0    60   Input ~ 0
+BUT2
+Text GLabel 1175 6800 0    60   Input ~ 0
+BUT2
+NoConn ~ 1175 6300
+Text GLabel 1175 6700 0    60   Input ~ 0
+BUT1
+NoConn ~ 2475 7000
+NoConn ~ 1175 5800
 $EndSCHEMATC

Commit message: update PCB
Connections:
- net BUT1: now also U2.45 (PB8); no longer U2.25 (PB12)
- net BUT2: now also U2.46 (PB9); no longer U2.26 (PB13)
- net Detec: now also U2.19 (PB1); no longer U2.14 (PA4)
- net LED_DATA_EN: now also U2.14 (PA4); no longer U2.31 (PA10)
- net col0: now also U2.22 (PB11); no longer U2.21 (PB10)
- net col1: now also U2.21 (PB10); no longer U2.41 (PB5)
- net col2: now also U2.20 (PB2); no longer U2.22 (PB11)
Changed lines of the file:
@@
 	4600 800  4800 800
-$Comp
-L MCU_ST_STM32F0:STM32F072C8Tx U2
-U 1 1 5E89A0AA
-P 1875 5700
-F 0 "U2" H 1875 5825 50  0000 C CNN
-F 1 "STM32F072C8Tx" H 1875 5675 50  0000 C CNN
-F 2 "Package_QFP:LQFP-48_7x7mm_P0.5mm" H 1275 4300 50  0001 R CNN
-F 3 "http://www.st.com/st-web-ui/static/active/en/resource/technical/document/datasheet/DM00090510.pdf" H 1875 5700 50  0001 C CNN
-	1    1875 5700
-	1    0    0    -1
-$EndComp
-Wire Wire Line
-	1775 4200 1875 4200
-Wire Wire Line
-	1875 4200 1975 4200
-Connection ~ 1875 4200
-Wire Wire Line
-	1975 4200 2075 4200
-Connection ~ 1975 4200
 $Comp
 L power:+3.3V #PWR014
@@
 Wire Wire Line
 	2075 4200 2075 4075
-Connection ~ 2075 4200
 $Comp
 L power:GND #PWR012
@@
 Wire Wire Line
 	1675 4000 1675 4200
-Wire Wire Line
-	1675 7200 1775 7200
-Wire Wire Line
-	1975 7200 1875 7200
-Connection ~ 1775 7200
-Connection ~ 1875 7200
-Wire Wire Line
-	1875 7200 1775 7200
 $Comp
 L power:GND #PWR013
@@
 Wire Wire Line
 	1675 7200 1675 7300
-Connection ~ 1675 7200
 $Comp
 L Connector:Micro_SD_Card_Det J1
@@
 Text GLabel 5000 7375 0    50   Input ~ 0
 Detec
-Text GLabel 2475 5900 2    50   Input ~ 0
+Text GLabel 1175 5600 0    50   Input ~ 0
 Detec
 Text GLabel 5000 6675 0    50   Input ~ 0
@@
 Text GLabel 2475 5500 2    60   Input ~ 0
 TIM2_CH1
+Text GLabel 1175 6600 0    60   Input ~ 0
+col0
 Text GLabel 1175 6500 0    60   Input ~ 0
-col0
-Text GLabel 1175 6000 0    60   Input ~ 0
 col1
-Text GLabel 1175 6600 0    60   Input ~ 0
+Text GLabel 1175 5700 0    60   Input ~ 0
 col2
 Text GLabel 2900 3900 2    50   Input ~ 0
@@
 Text GLabel 2475 6400 2    50   Input ~ 0
 UART1_TX
-Text GLabel 2475 6500 2    50   Input ~ 0
+Text GLabel 2475 5900 2    50   Input ~ 0
 LED_DATA_EN
 $Comp
@@
 	1    0    0    -1
 $EndComp
-NoConn ~ 1175 5700
-NoConn ~ 1175 5600
-NoConn ~ 1175 6400
 NoConn ~ 12950 150
 Wire Wire Line
@@
 Text GLabel 3275 6275 0    60   Input ~ 0
 BUT2
-Text GLabel 1175 6800 0    60   Input ~ 0
+Text GLabel 1175 6400 0    60   Input ~ 0
 BUT2
-NoConn ~ 1175 6300
-Text GLabel 1175 6700 0    60   Input ~ 0
+Text GLabel 1175 6300 0    60   Input ~ 0
 BUT1
+NoConn ~ 1175 5800
+NoConn ~ 1175 6800
+NoConn ~ 1175 6700
+Wire Wire Line
+	1975 4200 2075 4200
+Connection ~ 1975 4200
+Wire Wire Line
+	1875 4200 1975 4200
+Wire Wire Line
+	1775 4200 1875 4200
+Connection ~ 1875 4200
+Wire Wire Line
+	1975 7200 1875 7200
+Connection ~ 1875 7200
+Connection ~ 2075 4200
+Wire Wire Line
+	1875 7200 1775 7200
+Wire Wire Line
+	1675 7200 1775 7200
+Connection ~ 1775 7200
+Connection ~ 1675 7200
+$Comp
+L MCU_ST_STM32F0:STM32F072C8Tx U2
+U 1 1 5E89A0AA
+P 1875 5700
+F 0 "U2" H 1875 5825 50  0000 C CNN
+F 1 "STM32F072C8Tx" H 1875 5675 50  0000 C CNN
+F 2 "Package_QFP:LQFP-48_7x7mm_P0.5mm" H 1275 4300 50  0001 R CNN
+F 3 "http://www.st.com/st-web-ui/static/active/en/resource/technical/document/datasheet/DM00090510.pdf" H 1875 5700 50  0001 C CNN
+	1    1875 5700
+	1    0    0    -1
+$EndComp
+NoConn ~ 2475 6500
 NoConn ~ 2475 7000
-NoConn ~ 1175 5800
+NoConn ~ 1175 6000
 $EndSCHEMATC
