File: NumPad.kicad_pcb (KiCad board)
At the start: 2 copper layers, 120.1 x 132.9 mm, 112 parts, among them J1 Micro_SD_Card_Det, J2 OLED1, J3 OLED2, J4 Conn_01x05_Female, SW1 SW_SPST, SW10 SW_SPST, SW11 SW_SPST, SW12 SW_SPST, SW13 SW_SPST, SW14 SW_SPST, SW15 SW_SPST, SW16 SW_SPST, SW17 SW_SPST, SW18 SW_SPST, SW19 SW_SPST, SW2 SW_SPST, SW20 SW_SPST, SW21 SW_SPST, SW22 SW_SPST, SW23 SW_SPST, SW24 SW_SPST, SW25 SW_BUTTONRESET, SW26 SW_BUTTON2, SW27 SW_BUTTON1, SW28 SW_BOOT0, SW29 Rotary_Encoder_Switch, SW3 SW_SPST, SW4 SW_SPST, SW5 SW_SPST, SW6 SW_SPST, SW7 SW_SPST, SW8 SW_SPST, SW9 SW_SPST, U1 LM117_TO3, U2 STM32F072C8Tx, U3 74AHCT1G08

Commit message: update PCB
Parts:
- R4, R5, R8, R9: moved to B.Cu
- moved J4 107.9 mm to (137.9, 72.7)
- moved C6 58.1 mm to (116.6, 67.7), turned to 180 degrees
- moved SW28 57.5 mm to (143.7, 87.9), turned to 180 degrees
- moved SW25 49.5 mm to (143.7, 78.6), turned to 0 degrees
- moved R6 45.8 mm to (136.9, 89.1)
- moved R3 44.3 mm to (136.9, 79.8), turned to 270 degrees
- moved C5 44.0 mm to (110.1, 80.5), turned to 0 degrees
- moved U2 43.5 mm to (117.5, 74.8), turned to 45 degrees
- moved J1 39.9 mm to (103.6, 56.8), turned to 180 degrees
- moved C4 39.5 mm to (125.0, 73.2)
- moved C3 35.1 mm to (117.5, 82.3), turned to 180 degrees
- moved C1 20.2 mm to (131.2, 54.9), turned to 0 degrees
- moved R4 19.7 mm to (131.4, 88.2), turned to 180 degrees
- moved R10 18.3 mm to (91.4, 55.2), turned to 0 degrees
- moved U3 17.8 mm to (86.5, 65.8), turned to 180 degrees
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Connections:
- D49 pad 2: Net-(D49-Pad2) -> (no net)
- J1 pad 1: Net-(J1-Pad1) -> (no net)
- J1 pad 8: Net-(J1-Pad8) -> (no net)
- J1 pad 9: Net-(J1-Pad9) -> (no net)
- U2 pad 14: Detec -> LED_DATA_EN
- U2 pad 19: Net-(U2-Pad19) -> Detec
- U2 pad 20: Net-(U2-Pad20) -> col2
- U2 pad 21: col0 -> col1
- U2 pad 22: col2 -> col0
- U2 pad 25: BUT1 -> (no net)
- U2 pad 26: BUT2 -> (no net)
- U2 pad 29: Net-(U2-Pad29) -> (no net)
- U2 pad 31: LED_DATA_EN -> (no net)
- U2 pad 38: Net-(U2-Pad38) -> (no net)
- U2 pad 39: Net-(U2-Pad39) -> (no net)
- U2 pad 40: Net-(U2-Pad40) -> (no net)
- U2 pad 41: col1 -> (no net)
- U2 pad 45: Net-(U2-Pad45) -> BUT1
- U2 pad 46: Net-(U2-Pad46) -> BUT2
- USB1 pad 3: Net-(USB1-Pad3) -> (no net)
- USB1 pad 9: Net-(USB1-Pad9) -> (no net)
Routing:
- net +3V3: track 335.9 -> 262.9 mm, vias 9 -> 4
- net col1: track 238.1 -> 167.3 mm
- net USB_DP: track 76.0 -> 20.9 mm, vias 2 -> 0
- net col0: track 192.2 -> 246.8 mm
- net USB_DN: track 76.7 -> 22.7 mm, vias 2 -> 0
- net GND: track 528.2 -> 578.4 mm, vias 15 -> 11
- net POT_SLIDER: track 110.3 -> 62.3 mm
- net SYS_SWCLK: track 63.7 -> 16.8 mm
- net SYS_SWDIO: track 66.6 -> 19.9 mm, vias 0 -> 1
- net UART1_TX: track 69.4 -> 24.4 mm, vias 0 -> 1
- net row5: track 122.2 -> 164.3 mm
- net row4: track 103.7 -> 145.4 mm
- net row3: track 85.9 -> 127.1 mm
- net ENC_SWITCH: track 98.8 -> 57.7 mm
- net TIM2_CH2: track 74.0 -> 38.0 mm, vias 1 -> 2
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Other:
- outline, holes or cut-outs redrawn
- net class Default: clearance 0.2 -> 0.15
- net class power: clearance 0.2 -> 0.15
- rule trace_clearance: 0.2 -> 0.15

Commit message: Update PCB
Routing:
- net GND: track 578.4 -> 579.2 mm
Other:
- board size 120.1 x 132.9 mm -> 143.4 x 132.9 mm
Changed lines of the file:
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@@
   (general
     (thickness 1.6)
-    (drawings 105)
-    (tracks 1090)
+    (drawings 107)
+    (tracks 1093)
     (zones 0)
     (modules 112)
@@
       (net 84 GND))
   )
-  (gr_line (start 19.9 183.675) (end 140 183.675) (layer Edge.Cuts) (width 0.05))
+  (gr_line (start 163.325 50.8) (end 163.325 183.675) (layer Edge.Cuts) (width 0.05))
+  (gr_line (start 19.9 50.8) (end 163.325 50.8) (layer Edge.Cuts) (width 0.05))
+  (gr_line (start 19.9 183.675) (end 163.325 183.675) (layer Edge.Cuts) (width 0.05))
   (gr_line (start 19.9 50.8) (end 19.9 183.675) (layer Edge.Cuts) (width 0.05))
   (gr_line (start 102.39 138.9) (end 137.99 138.9) (layer Dwgs.User) (width 0.15))
@@
   (segment (start 90.225 60.95) (end 90.625 61.35) (width 0.25) (layer B.Cu) (net 59))
   (segment (start 86.875 60.95) (end 90.225 60.95) (width 0.25) (layer B.Cu) (net 59))
-  (segment (start 109.775 78.325) (end 109.775 78.325) (width 0.25) (layer F.Cu) (net 59))
-  (via (at 109.775 78.325) (size 0.6) (drill 0.4) (layers F.Cu B.Cu) (net 59))
-  (segment (start 111.538462 78.325) (end 113.345569 76.517893) (width 0.25) (layer B.Cu) (net 59))
-  (segment (start 109.775 78.325) (end 111.538462 78.325) (width 0.25) (layer B.Cu) (net 59))
   (via (at 105.075 74.475) (size 0.6) (drill 0.4) (layers F.Cu B.Cu) (net 59))
   (segment (start 103.275 74.475) (end 105.075 74.475) (width 0.25) (layer B.Cu) (net 59))
   (segment (start 90.625 61.35) (end 90.625 61.825) (width 0.25) (layer B.Cu) (net 59))
   (segment (start 90.625 61.825) (end 103.275 74.475) (width 0.25) (layer B.Cu) (net 59))
-  (segment (start 108.925 78.325) (end 109.775 78.325) (width 0.25) (layer F.Cu) (net 59))
-  (segment (start 105.075 74.475) (end 108.925 78.325) (width 0.25) (layer F.Cu) (net 59))
+  (segment (start 108.925 78.325) (end 105.075 74.475) (width 0.25) (layer F.Cu) (net 59))
+  (segment (start 109.25 78.325) (end 108.925 78.325) (width 0.25) (layer F.Cu) (net 59))
+  (segment (start 111.538462 78.325) (end 113.345569 76.517893) (width 0.25) (layer B.Cu) (net 59))
+  (via (at 109.25 78.325) (size 0.6) (drill 0.4) (layers F.Cu B.Cu) (net 59))
+  (segment (start 109.25 78.325) (end 111.538462 78.325) (width 0.25) (layer B.Cu) (net 59))
   (segment (start 109.625 77.625) (end 109.625 77.625) (width 0.25) (layer F.Cu) (net 60))
   (via (at 109.625 77.625) (size 0.6) (drill 0.4) (layers F.Cu B.Cu) (net 60))
@@
   (via (at 116.25 62.575) (size 0.6) (drill 0.4) (layers F.Cu B.Cu) (net 84))
   (segment (start 116.52755 82.12755) (end 116.52755 82.12755) (width 0.2) (layer B.Cu) (net 84))
-  (via (at 119.4 81.025) (size 0.6) (drill 0.4) (layers F.Cu B.Cu) (net 84))
-  (segment (start 119.4 79.86764) (end 119.4 81.025) (width 0.2) (layer B.Cu) (net 84))
-  (segment (start 118.87868 79.34632) (end 119.4 79.86764) (width 0.2) (layer B.Cu) (net 84))
+  (segment (start 119.4 79.86764) (end 118.87868 79.34632) (width 0.2) (layer B.Cu) (net 84))
+  (via (at 119.475 81.075) (size 0.6) (drill 0.4) (layers F.Cu B.Cu) (net 84))
+  (segment (start 118.87868 79.34632) (end 119.475 79.94264) (width 0.2) (layer B.Cu) (net 84))
+  (segment (start 119.475 79.94264) (end 119.475 81.075) (width 0.2) (layer B.Cu) (net 84))
   (segment (start 119.95 79.710534) (end 119.232233 78.992767) (width 0.25) (layer B.Cu) (net 85))
-  (segment (start 119.95 82.6875) (end 119.95 79.710534) (width 0.25) (layer B.Cu) (net 85))
   (segment (start 114.7125 87.925) (end 119.95 82.6875) (width 0.25) (layer B.Cu) (net 85))
   (segment (start 114.7125 88.4) (end 114.7125 87.925) (width 0.25) (layer B.Cu) (net 85))
@@
   (via (at 114.595 90.225) (size 0.6) (drill 0.4) (layers F.Cu B.Cu) (net 85))
   (segment (start 114.7125 88.4) (end 114.595 90.225) (width 0.25) (layer B.Cu) (net 85))
+  (segment (start 119.95 82.6875) (end 119.95 82.675) (width 0.25) (layer B.Cu) (net 85))
+  (segment (start 119.95 82.675) (end 120.275 82.35) (width 0.25) (layer B.Cu) (net 85))
+  (segment (start 120.275 80.035534) (end 119.95 79.710534) (width 0.25) (layer B.Cu) (net 85))
+  (segment (start 120.275 82.35) (end 120.275 80.035534) (width 0.25) (layer B.Cu) (net 85))
   (zone (net 84) (net_name GND) (layer B.Cu) (hatch edge 0.508)
     (connect_pads (clearance 0.2))

Commit message: Update
Parts:
- moved J1 0.48 mm to (103.7, 57.3)
Routing:
- net GND: track 579.2 -> 564.2 mm, vias 11 -> 13
- net SPI_MISO: track 29.1 -> 27.7 mm
Changed lines of the file:
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@@
     (thickness 1.6)
     (drawings 107)
-    (tracks 1093)
+    (tracks 1089)
     (zones 0)
     (modules 112)
@@
   )
   (module Connector_Card:microSD_HC_Molex_104031-0811 (layer B.Cu)
-    (at 103.625 56.825 180)
+    (at 103.68 57.3 180)
     (descr "1.10mm Pitch microSD Memory Card Connector, Surface Mount, Push-Pull Type, 1.42mm Height, with Detect Switch (https://www.molex.com/pdm_docs/sd/1040310811_sd.pdf)")
     (tags "microSD SD molex")
@@
   (gr_line (start 137.99 138.9) (end 137.99 172.4) (layer Dwgs.User) (width 0.15))
   (gr_line (start 102.39 138.9) (end 102.39 172.4) (layer Dwgs.User) (width 0.15))
+  (via (at 97.925 51.75) (size 0.6) (drill 0.4) (layers F.Cu B.Cu) (net 84))
   (segment (start 91.05 83.335) (end 91.05 82.725) (width 0.2) (layer B.Cu) (net 1))
   (segment (start 72 83.335) (end 72 82.725) (width 0.2) (layer B.Cu) (net 1))
@@
   (segment (start 117.5 68.951672) (end 117.5 67.725) (width 0.25) (layer B.Cu) (net 2))
   (segment (start 116.52755 69.924122) (end 117.5 68.951672) (width 0.25) (layer B.Cu) (net 2))
-  (via (at 103.425 51.35) (size 0.6) (drill 0.4) (layers F.Cu B.Cu) (net 2))
-  (segment (start 103.425 51.774264) (end 103.425 51.35) (width 0.38) (layer F.Cu) (net 2))
-  (segment (start 104.525736 52.875) (end 103.425 51.774264) (width 0.38) (layer F.Cu) (net 2))
-  (segment (start 122.85 52.875) (end 104.525736 52.875) (width 0.38) (layer F.Cu) (net 2))
-  (segment (start 128.225 58.25) (end 122.85 52.875) (width 0.38) (layer F.Cu) (net 2))
   (via (at 129.825 63.325) (size 0.6) (drill 0.4) (layers F.Cu B.Cu) (net 2))
-  (segment (start 128.225 61.725) (end 129.825 63.325) (width 0.38) (layer F.Cu) (net 2))
-  (segment (start 128.225 58.25) (end 128.225 61.725) (width 0.38) (layer F.Cu) (net 2))
-  (segment (start 101.9 52.875) (end 103.425 51.35) (width 0.38) (layer F.Cu) (net 2))
-  (segment (start 92.2 55.2) (end 94.5 52.875) (width 0.38) (layer F.Cu) (net 2))
-  (segment (start 94.5 52.875) (end 101.9 52.875) (width 0.38) (layer F.Cu) (net 2))
   (via (at 92.2 55.2) (size 0.6) (drill 0.4) (layers F.Cu B.Cu) (net 2))
   (segment (start 92.2 55.2) (end 92.2 55.175) (width 0.38) (layer B.Cu) (net 2))
@@
   (segment (start 135.425 91.875) (end 132.175 88.625) (width 0.38) (layer B.Cu) (net 2))
   (segment (start 141.95 91.875) (end 135.425 91.875) (width 0.38) (layer B.Cu) (net 2))
+  (segment (start 102.46 52.875) (end 103.485 51.85) (width 0.38) (layer F.Cu) (net 2))
+  (segment (start 94.5 52.875) (end 102.46 52.875) (width 0.38) (layer F.Cu) (net 2))
+  (segment (start 92.2 55.2) (end 94.5 52.875) (width 0.38) (layer F.Cu) (net 2))
+  (via (at 103.485 51.85) (size 0.6) (drill 0.4) (layers F.Cu B.Cu) (net 2))
+  (segment (start 103.485 52.16) (end 104.2 52.875) (width 0.38) (layer F.Cu) (net 2))
+  (segment (start 122.85 52.875) (end 128.225 58.25) (width 0.38) (layer F.Cu) (net 2))
+  (segment (start 128.225 61.725) (end 129.825 63.325) (width 0.38) (layer F.Cu) (net 2))
+  (segment (start 103.485 51.85) (end 103.485 52.16) (width 0.38) (layer F.Cu) (net 2))
+  (segment (start 104.2 52.875) (end 122.85 52.875) (width 0.38) (layer F.Cu) (net 2))
+  (segment (start 128.225 58.25) (end 128.225 61.725) (width 0.38) (layer F.Cu) (net 2))
   (segment (start 119.535 59.08) (end 119.535 57.655) (width 0.2) (layer B.Cu) (net 3))
   (segment (start 119.434999 59.180001) (end 119.535 59.08) (width 0.2) (layer B.Cu) (net 3))
@@
   (segment (start 102.331734 62.092268) (end 102.331734 55.318266) (width 0.25) (layer B.Cu) (net 45))
   (segment (start 113.345569 73.106103) (end 102.331734 62.092268) (width 0.25) (layer B.Cu) (net 45))
-  (segment (start 100.13 51.949332) (end 100.13 51.375) (width 0.2) (layer B.Cu) (net 46))
-  (segment (start 100.13 52.268002) (end 100.13 51.375) (width 0.2) (layer B.Cu) (net 46))
   (segment (start 100.13 52.175) (end 100.13 51.375) (width 0.25) (layer B.Cu) (net 46))
   (segment (start 100.13 52.330002) (end 100.13 52.175) (width 0.25) (layer B.Cu) (net 46))
@@
   (segment (start 107.564979 66.614979) (end 107.115001 66.165001) (width 0.25) (layer B.Cu) (net 46))
   (segment (start 107.115001 58.259999) (end 107.125 58.25) (width 0.2) (layer B.Cu) (net 46))
-  (segment (start 107.115001 66.165001) (end 107.115001 58.259999) (width 0.25) (layer B.Cu) (net 46))
   (segment (start 107.125 58.25) (end 103.117879 54.225001) (width 0.25) (layer B.Cu) (net 46))
-  (segment (start 109.365 66.297106) (end 109.365 61.225) (width 0.25) (layer B.Cu) (net 47))
+  (segment (start 107.145001 66.135001) (end 107.145001 58.270001) (width 0.25) (layer B.Cu) (net 46))
+  (segment (start 107.145001 58.270001) (end 107.125 58.25) (width 0.25) (layer B.Cu) (net 46))
+  (segment (start 107.115001 66.165001) (end 107.145001 66.135001) (width 0.25) (layer B.Cu) (net 46))
   (segment (start 114.759783 71.691889) (end 109.365 66.297106) (width 0.25) (layer B.Cu) (net 47))
+  (segment (start 109.42 66.242106) (end 109.42 61.7) (width 0.25) (layer B.Cu) (net 47))
+  (segment (start 109.365 66.297106) (end 109.42 66.242106) (width 0.25) (layer B.Cu) (net 47))
   (segment (start 118.5 142.73) (end 118.43 142.8) (width 0.25) (layer F.Cu) (net 48))
   (segment (start 118.43 142.8) (end 118.43 142.77) (width 0.25) (layer F.Cu) (net 48))
@@
   (segment (start 131.925 59.557002) (end 132.65 58.832002) (width 0.38) (layer B.Cu) (net 84))
   (segment (start 131.925 60.45) (end 131.925 59.557002) (width 0.38) (layer B.Cu) (net 84))
-  (segment (start 101.23 50.445) (end 101.23 51.375) (width 0.38) (layer B.Cu) (net 84))
-  (segment (start 101.219999 50.434999) (end 101.23 50.445) (width 0.38) (layer B.Cu) (net 84))
-  (segment (start 98.392999 50.434999) (end 101.219999 50.434999) (width 0.38) (layer B.Cu) (net 84))
-  (segment (start 97.87 50.957998) (end 98.392999 50.434999) (width 0.38) (layer B.Cu) (net 84))
-  (segment (start 97.87 51.725) (end 97.87 50.957998) (width 0.38) (layer B.Cu) (net 84))
-  (segment (start 109.19 50.445) (end 109.19 51.5) (width 0.38) (layer B.Cu) (net 84))
-  (segment (start 109.179999 50.434999) (end 109.19 50.445) (width 0.38) (layer B.Cu) (net 84))
-  (segment (start 101.592999 50.434999) (end 109.179999 50.434999) (width 0.38) (layer B.Cu) (net 84))
-  (segment (start 101.23 50.797998) (end 101.592999 50.434999) (width 0.38) (layer B.Cu) (net 84))
-  (segment (start 101.23 51.375) (end 101.23 50.797998) (width 0.38) (layer B.Cu) (net 84))
   (segment (start 114.28 51.5) (end 114.455 51.325) (width 0.38) (layer B.Cu) (net 84))
   (segment (start 109.19 51.5) (end 114.28 51.5) (width 0.38) (layer B.Cu) (net 84))
@@
   (segment (start 118.87868 79.34632) (end 119.475 79.94264) (width 0.2) (layer B.Cu) (net 84))
   (segment (start 119.475 79.94264) (end 119.475 81.075) (width 0.2) (layer B.Cu) (net 84))
+  (segment (start 101.285 51.85) (end 101.225 51.85) (width 0.38) (layer B.Cu) (net 84))
+  (segment (start 101.225 51.85) (end 101.23 51.845) (width 0.38) (layer B.Cu) (net 84))
+  (segment (start 101.225 51.85) (end 101.225 51.85) (width 0.38) (layer B.Cu) (net 84))
+  (via (at 101.225 51.85) (size 0.6) (drill 0.4) (layers F.Cu B.Cu) (net 84))
   (segment (start 119.95 79.710534) (end 119.232233 78.992767) (width 0.25) (layer B.Cu) (net 85))
   (segment (start 114.7125 87.925) (end 119.95 82.6875) (width 0.25) (layer B.Cu) (net 85))
