File: NumPad.kicad_pcb (KiCad board)
At the start: 2 copper layers, 143.4 x 132.9 mm, 112 parts, among them J1 Micro_SD_Card_Det, J2 OLED1, J3 OLED2, J4 Conn_01x05_Female, SW1 SW_SPST, SW10 SW_SPST, SW11 SW_SPST, SW12 SW_SPST, SW13 SW_SPST, SW14 SW_SPST, SW15 SW_SPST, SW16 SW_SPST, SW17 SW_SPST, SW18 SW_SPST, SW19 SW_SPST, SW2 SW_SPST, SW20 SW_SPST, SW21 SW_SPST, SW22 SW_SPST, SW23 SW_SPST, SW24 SW_SPST, SW25 SW_BUTTONRESET, SW26 SW_BUTTON2, SW27 SW_BUTTON1, SW28 SW_BOOT0, SW29 Rotary_Encoder_Switch, SW3 SW_SPST, SW4 SW_SPST, SW5 SW_SPST, SW6 SW_SPST, SW7 SW_SPST, SW8 SW_SPST, SW9 SW_SPST, U1 LM117_TO3, U2 STM32F072C8Tx, U3 74AHCT1G08

Commit message: update
Parts:
- moved R6 7.74 mm to (130.3, 85.0)
- moved J4 7.62 mm to (130.3, 72.6)
- moved SW25 7.31 mm to (136.4, 78.6)
- moved SW28 7.31 mm to (136.4, 87.9)
- moved R3 6.55 mm to (130.4, 79.8)
- moved SW26 4.96 mm to (106.7, 92.0)
- moved SW27 3.65 mm to (125.5, 92.0)
- moved R4 3.56 mm to (127.8, 88.3)
Routing:
- net +3V3: track 262.4 -> 249.3 mm
- net UART1_TX: track 24.4 -> 16.8 mm
- net SYS_SWDIO: track 19.9 -> 12.5 mm
- net Net-(R3-Pad2): track 28.5 -> 21.3 mm
- net GND: track 564.2 -> 571.2 mm, vias 13 -> 15
- net BOOT0: track 25.5 -> 18.9 mm
- net SYS_SWCLK: track 16.8 -> 10.5 mm
- net BUT2: track 14.1 -> 18.7 mm
- net BUT1: track 18.4 -> 16.6 mm
Other:
- board size 143.4 x 132.9 mm -> 122.6 x 133.5 mm
